File: hardware/teste_estatico/kicad/teste_estatico.kicad_pcb (KiCad board)
At the start: 2 copper layers, 11 parts, among them J1 Sensor de pressão, J2 sd card, J3 USB_A, U2 HX711-Mod

Commit message: adcionado arquivo para fabricação cnc
Parts:
- removed J1: Sensor de pressão, Connector_PinSocket_2.54mm:PinSocket_1x03_P2.54mm_Vertical
- removed J2: sd card, Connector_PinSocket_2.54mm:PinSocket_1x06_P2.54mm_Vertical
- removed J3: USB_A, Connector_USB:USB_A_CNCTech_1001-011-01101_Horizontal
- removed U2: HX711-Mod, HX711_mod:HX711_module
- added PRESSÃO1: Sensor de pressão, Connector_PinSocket_2.54mm:PinSocket_1x03_P2.54mm_Vertical, F.Cu at (144.3, 98.8)
- added RJ45: conexão do rj45, Connector_PinSocket_2.54mm:PinSocket_1x04_P2.54mm_Vertical, F.Cu at (139.7, 98.8)
- added SDCARD1: sd card, Connector_PinSocket_2.54mm:PinSocket_1x06_P2.54mm_Vertical, F.Cu at (139.7, 67.3)
- moved R3.3k1 86.7 mm to (138.9, 94.1)
- moved D1 84.0 mm to (144.5, 110.0)
- moved R2.2k1 72.9 mm to (138.9, 84.6)
- moved tara1 68.6 mm to (144.0, 75.5)
- moved R220ohn1 66.0 mm to (138.9, 89.4)
- moved A1 55.5 mm to (109.6, 76.2), turned to 0 degrees
- moved NOVOARQUIVO1 45.8 mm to (144.0, 67.0)
