File: hardware/teste_estatico/kicad/teste_estatico.kicad_pcb (KiCad board)
At the start: 2 copper layers, 10 parts

Commit message: adcionado atulização nos arquivos de pcb kicad
Routing:
- net Net-(A1-VIN): track 0.00 -> 294.5 mm
- net Net-(A1-D19): track 0.00 -> 188.1 mm
- net Net-(A1-ADC1_CH7/D35): track 89.0 -> 266.7 mm
- net Net-(PRESSÃO1-Pad1): track 0.00 -> 157.9 mm
- net Net-(A1-D23): track 0.00 -> 98.4 mm
- net Net-(A1-D4/ADC2_CH0): track 0.00 -> 95.6 mm
- net Net-(A1-DAC2/ADC2_CH9/D26): track 0.00 -> 82.3 mm
- net Net-(A1-ADC2_CH7/D27): track 0.00 -> 73.5 mm
- net Net-(A1-GND-Pad2): track 0.00 -> 56.2 mm
- net Net-(A1-D5): track 0.00 -> 55.9 mm
- net Net-(PRESSÃO1-Pad3): track 0.00 -> 55.6 mm
- net Net-(A1-ADC1_CH4/D32-Pad22): track 6.50 -> 62.1 mm
- net Net-(A1-RX2/GPIO16): track 0.00 -> 51.4 mm
- net Net-(A1-ADC1_CH4/D32-Pad21): track 6.50 -> 43.6 mm
- net Net-(D1-A): track 0.00 -> 18.8 mm
