File: hardware/teste_estatico/kicad/teste_estatico.kicad_sch (KiCad schematic)
At the start: 11 parts, among them J1 Sensor de pressão, J2 sd card, J3 USB_A, U2 HX711-Mod

Commit message: adcionado arquivo para fabricação cnc
Parts:
- removed J3: USB_A, Connector_USB:USB_A_CNCTech_1001-011-01101_Horizontal, symbol Connector:USB_A
- removed U2: HX711-Mod, HX711_module, symbol HX711_module:HX711_module
- added RJ45: conexão do rj45, Connector_PinSocket_2.54mm:PinSocket_1x04_P2.54mm_Vertical, symbol PCM_SL_Pin_Headers:PINHD_1x4_Female
- renumbered J1 to PRESSÃO1, J2 to SDCARD1
Connections:
- net at A1.20 (ADC1_CH7/D35), A1.29 (GND), NOVOARQUIVO1.2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: now also RJ45.1
- net at A1.24 (DAC2/ADC2_CH9/D26): now also RJ45.3
- net at A1.25 (ADC2_CH7/D27): now also RJ45.2
- net at A1.30 (VIN), PRESSÃO1.2, SDCARD1.2: now also RJ45.4
Other:
- note added: "CLK"
- note added: "DAT"
- note added: "VDD"

Commit message: atulização nos arquivos de pcb
Parts:
- removed SDCARD1: sd card, Connector_PinSocket_2.54mm:PinSocket_1x06_P2.54mm_Vertical, symbol PCM_SL_Pin_Headers:PINHD_1x6_Female
- added J1: SDK_GND, Connector_PinSocket_2.54mm:PinSocket_1x01_P2.54mm_Vertical, symbol PCM_SL_Pin_Headers:PINHD_1x1_Female
- added J2: SDK_VCC, Connector_PinSocket_2.54mm:PinSocket_1x01_P2.54mm_Vertical, symbol PCM_SL_Pin_Headers:PINHD_1x1_Female
- added J3: SDK_MISO, Connector_PinSocket_2.54mm:PinSocket_1x01_P2.54mm_Vertical, symbol PCM_SL_Pin_Headers:PINHD_1x1_Female
- added J4: SDK_MOSI, Connector_PinSocket_2.54mm:PinSocket_1x01_P2.54mm_Vertical, symbol PCM_SL_Pin_Headers:PINHD_1x1_Female
- added J5: SDK_SCK, Connector_PinSocket_2.54mm:PinSocket_1x01_P2.54mm_Vertical, symbol PCM_SL_Pin_Headers:PINHD_1x1_Female
- added J6: SDK_CK, Connector_PinSocket_2.54mm:PinSocket_1x01_P2.54mm_Vertical, symbol PCM_SL_Pin_Headers:PINHD_1x1_Female
Connections:
- net at A1.20 (ADC1_CH7/D35), A1.29 (GND), NOVOARQUIVO1.2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: now also J1.1
- net at A1.10 (D19): now also J3.1
- net at A1.15 (D23): now also J4.1
- net at A1.30 (VIN), PRESSÃO1.2, RJ45.4: now also J2.1
- net at A1.6 (RX2/GPIO16): now also J5.1
- net at A1.8 (D5): now also J6.1
