File: hardware/teste_estatico/kicad/projeto kicad/_restore_backup_2026-05-29T19-16-41-364/teste_estatico.kicad_sch (KiCad schematic)
At the start: 15 parts, among them J1 SDK_GND, J2 SDK_VCC, J3 SDK_MISO, J4 SDK_MOSI, J5 SDK_SCK, J6 SDK_CK

Commit message: feat: adcionado arquivos de fabricação e modificação na pcb
Parts:
- renumbered R3.3k1 to R2.2k1, R2.2k1 to R3.3k1
