File: hardware/teste_estatico/kicad/projeto kicad/teste_estatico.kicad_pcb (KiCad board)
At the start: 2 copper layers, 10 parts, among them J1 PINHD_1x6_Female

Commit message: chore: atualizando a pcb
Parts:
- removed NOVOARQUIVO1: Push_Button, Button_Switch_THT:SW_PUSH_6mm
- added BZ1: Buzzer_5V, Buzzer_Beeper:MagneticBuzzer_ProSignal_ABT-410-RC, F.Cu at (136.2, 102.0)
- added J2: PINHD_1x2_Female, Connector_PinSocket_2.54mm:PinSocket_1x02_P2.54mm_Vertical, F.Cu at (160.6, 82.5)
- A1, D1, R220ohn1, RJ45, tara1: moved to B.Cu
- J1: footprint PCM_SL_Connectors:PinSocket_1x06_P2.54mm_Vertical -> Connector_PinSocket_2.54mm:PinSocket_1x06_P2.54mm_Vertical
- R2.2k1: renamed from R3.3k1; moved to B.Cu
- R3.3k1: renamed from R2.2k1; moved to B.Cu
- sensor2: renamed from PRESSÃO1; moved to B.Cu
- moved R2.2k1 91.9 mm to (105.2, 113.5), turned to -90 degrees
- moved sensor2 82.7 mm to (120.7, 117.8)
- moved J1 81.1 mm to (168.8, 120.2), turned to -90 degrees
- moved A1 64.9 mm to (174.5, 76.2), turned to 180 degrees
- moved D1 62.1 mm to (173.1, 126.8), turned to 180 degrees
- moved tara1 58.9 mm to (112.6, 97.5), turned to 180 degrees
- moved RJ45 40.4 mm to (121.8, 73.5)
- moved R3.3k1 30.9 mm to (126.6, 126.2), turned to 180 degrees
- moved R220ohn1 19.5 mm to (151.8, 126.8), turned to 180 degrees
Connections:
- A1 pad 1: unconnected-(A1-3.3V-Pad1) -> 3.3V
- A1 pad 2: Net-(A1-GND-Pad2) -> GND
- A1 pad 23: unconnected-(A1-DAC1/ADC2_CH8/D25-Pad23) -> Net-(A1-DAC1/ADC2_CH8/D25)
- A1 pad 24: Net-(A1-DAC2/ADC2_CH9/D26) -> unconnected-(A1-DAC2/ADC2_CH9/D26-Pad24)
- A1 pad 30: Net-(A1-VIN) -> VIN
- A1 pad 6: Net-(A1-RX2/GPIO16) -> unconnected-(A1-RX2/GPIO16-Pad6)
- A1 pad 9: unconnected-(A1-D18-Pad9) -> Net-(A1-D18)
- D1 pad 1: Net-(A1-D4/ADC2_CH0) -> Net-(A1-D19)
- J1 pad 1: Net-(A1-GND-Pad2) -> 3.3V
- J1 pad 2: Net-(A1-VIN) -> Net-(A1-D5)
- J1 pad 3: Net-(A1-D19) -> Net-(A1-ADC2_CH7/D27)
- J1 pad 4: Net-(A1-D23) -> Net-(A1-DAC1/ADC2_CH8/D25)
- J1 pad 5: Net-(A1-RX2/GPIO16) -> Net-(A1-D23)
- J1 pad 6: Net-(A1-D5) -> GND
- R2.2k1 pad 1: Net-(PRESSÃO1-Pad3) -> Net-(R2.2k1-Pad1)
- RJ45 pad 1: Net-(A1-ADC1_CH7/D35) -> GND
- RJ45 pad 2: Net-(A1-ADC2_CH7/D27) -> Net-(A1-D18)
- RJ45 pad 3: Net-(A1-DAC2/ADC2_CH9/D26) -> Net-(A1-D4/ADC2_CH0)
- RJ45 pad 4: Net-(A1-VIN) -> 3.3V
- sensor2 pad 2: Net-(A1-VIN) -> VIN
Routing:
- net Net-(A1-VIN): track 224.7 -> 0.00 mm
- net GND: track 0.00 -> 214.1 mm
- net VIN: track 0.00 -> 183.1 mm
- net Net-(A1-D18): track 0.00 -> 158.1 mm
- net Net-(R3.3k1-Pad1): track 157.9 -> 10.9 mm
- net Net-(A1-ADC1_CH7/D35): track 266.7 -> 127.6 mm
- net 3.3V: track 0.00 -> 108.3 mm
- net Net-(A1-DAC2/ADC2_CH9/D26): track 82.3 -> 0.00 mm
- net Net-(A1-D4/ADC2_CH0): track 61.8 -> 126.8 mm
- net Net-(PRESSÃO1-Pad3): track 55.6 -> 0.00 mm
- net Net-(A1-D19): track 83.3 -> 35.2 mm
- net Net-(A1-ADC2_CH7/D27): track 73.5 -> 38.3 mm
- net Net-(A1-DAC1/ADC2_CH8/D25): track 0.00 -> 32.2 mm
- net Net-(A1-ADC1_CH4/D32-Pad21): track 43.6 -> 14.1 mm
- net Net-(A1-GND-Pad2): track 19.8 -> 0.00 mm
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Other:
- board outline added: 92.1 x 81.2 mm

Commit message: chore: atualizando a pcb
Routing:
- net VIN: track 183.1 -> 179.8 mm
- net Net-(A1-ADC1_CH7/D35): track 127.6 -> 124.8 mm
- net GND: track 214.1 -> 215.7 mm
- net Net-(A1-D18): track 158.1 -> 156.8 mm
- net Net-(A1-D4/ADC2_CH0): track 126.8 -> 125.6 mm
- net Net-(A1-D19): track 35.2 -> 34.4 mm
- net 3.3V: track 108.3 -> 107.7 mm
